Commit message: wheel controller

File: src/mulinex_description/urdf/track.xacro (robot description, xacro)
@@ -41,5 +41,5 @@
       <child link="${name}"/>
       <axis xyz="0 0 1"/>
-      <limit effort="10" velocity="10"/>
+      <limit effort="10" velocity="100000"/>
     </joint>
   </xacro:macro>
@@ -51,5 +51,5 @@
       <child link="${name}"/>
       <axis xyz="1 0 0"/>
-      <limit effort="10" velocity="10" lower="-0.785398" upper="0.785398"/>
+      <limit effort="10" velocity="10" lower="-3.14159" upper="3.14159"/>
     </joint>
     <link name="${name}">
