Commit message: Fix traquad track description for Gazebo
- traquad.xacro: remove duplicated track bodies/wheels (already
  instantiated in track.xacro); the duplicates doubled mass/collisions
  and their wheel joints were not controlled.
- track.xacro: limit the passive ankle joint to +-0.35 rad around the
  flat-track pose (+-0.441 rad) and add damping, so tracks no longer
  flip over when driven.
- track.xacro: wheel collision as a cylinder (r=0.015, w=0.045)
  instead of the mesh, since DART ignores friction params on the mesh;
  anisotropic friction (lateral mu=0.1, longitudinal mu2=1.0) so the
  skid-steer robot can yaw.

Tested in Gazebo Fortress: v=0.2 m/s, w=+-0.3 rad/s tracked with
effective track width 0.395 m, wheel radius 0.015 m.

File: src/mulinex_description/urdf/track.xacro (robot description, xacro)
@@ -7,5 +7,14 @@
   <xacro:property name="wheel_izz" default="1.15625e-05"/>
   <xacro:property name="wheel_mesh" default="file://$(find mulinex_description)/meshes//wheel.stl"/>
+  <!-- Gazebo-only wheel friction: reduced lateral friction lets the skid-steer tracks turn.
+       mu acts along fdir1 (= wheel axis, lateral), mu2 along the rolling direction. -->
+  <xacro:property name="wheel_mu_lat" value="0.1"/>
+  <xacro:property name="wheel_mu_long" value="1.0"/>
   <xacro:property name="body_mass" value="0.6"/>
+  <!-- Passive ankle: range centred on the pose where the track lies flat
+       (wheels 1-3 level) with HFE at init_pos (+-1.13 rad) -->
+  <xacro:property name="ankle_flat" value="0.441"/>
+  <xacro:property name="ankle_range" value="0.35"/>
+  <xacro:property name="ankle_damping" value="0.05"/>
   <xacro:property name="body_left_mesh" default="file://$(find mulinex_description)/meshes//body_left.stl"/>
   <xacro:property name="body_right_mesh" default="file://$(find mulinex_description)/meshes//body_right.stl"/>
@@ -30,7 +39,8 @@
       </visual>
       <collision>
-        <origin xyz="0 0 -0.045" rpy="-1.5708 -1.5708 0"/>
+        <!-- primitive equivalent of wheel.stl (r=0.015, width=0.045), friction params are applied to it -->
+        <origin xyz="0 0 -0.0225" rpy="0 0 0"/>
         <geometry>
-          <mesh filename="${wheel_mesh}"/>
+          <cylinder radius="0.015" length="0.045"/>
         </geometry>
       </collision>
@@ -43,7 +53,21 @@
       <limit effort="10" velocity="100000"/>
     </joint>
+    <gazebo reference="${name}">
+      <collision>
+        <surface>
+          <friction>
+            <ode>
+              <mu>${wheel_mu_lat}</mu>
+              <mu2>${wheel_mu_long}</mu2>
+              <!-- wheel axis (joint axis, link z) -->
+              <fdir1>0 0 1</fdir1>
+            </ode>
+          </friction>
+        </surface>
+      </collision>
+    </gazebo>
   </xacro:macro>
   <!-- Macro CORPO LEFT -->
-  <xacro:macro name="body_left" params="name parent xyz rpy">
+  <xacro:macro name="body_left" params="name parent xyz rpy ankle_center">
     <joint name="${name}_ankle" type="revolute">
       <origin xyz="${xyz}" rpy="${rpy}"/>
@@ -51,5 +75,6 @@
       <child link="${name}"/>
       <axis xyz="1 0 0"/>
-      <limit effort="10" velocity="10" lower="-3.14159" upper="3.14159"/>
+      <limit effort="10" velocity="10" lower="${ankle_center - ankle_range}" upper="${ankle_center + ankle_range}"/>
+      <dynamics damping="${ankle_damping}" friction="0.0"/>
     </joint>
     <link name="${name}">
@@ -78,5 +103,5 @@
   </xacro:macro>
   <!-- Macro CORPO RIGHT -->
-  <xacro:macro name="body_right" params="name parent xyz rpy">
+  <xacro:macro name="body_right" params="name parent xyz rpy ankle_center">
     <joint name="${name}_ankle" type="revolute">
       <origin xyz="${xyz}" rpy="${rpy}"/>
@@ -84,5 +109,6 @@
       <child link="${name}"/>
       <axis xyz="1 0 0"/>
-      <limit effort="10" velocity="10" lower="-3.14159" upper="3.14159"/>
+      <limit effort="10" velocity="10" lower="${ankle_center - ankle_range}" upper="${ankle_center + ankle_range}"/>
+      <dynamics damping="${ankle_damping}" friction="0.0"/>
     </joint>
     <link name="${name}">
@@ -113,5 +139,5 @@
   <!-- LEFT_H -->
   <xacro:body_left name="body_left_H" parent="LH_UPPER_LEG"
-                   xyz="-0.19 0.05 0" rpy="1.5708 0 1.5708"/>
+                   xyz="-0.19 0.05 0" rpy="1.5708 0 1.5708" ankle_center="${-ankle_flat}"/>
   <xacro:wheel name="wheel_1_LEFT_H" parent="body_left_H" xyz="0 0.0484063 -0.0583795" rpy="-6.12323e-17 -1.5708 0"/>
   <xacro:wheel name="wheel_2_LEFT_H" parent="body_left_H" xyz="0 1.07779e-16 -0.0583795" rpy="-6.12323e-17 -1.5708 0"/>
@@ -120,5 +146,5 @@
   <!-- LEFT_F -->
   <xacro:body_left name="body_left_F" parent="LF_UPPER_LEG"
-                   xyz="0.19 0.05 0" rpy="-1.5708 0 1.5708"/>
+                   xyz="0.19 0.05 0" rpy="-1.5708 0 1.5708" ankle_center="${ankle_flat}"/>
   <xacro:wheel name="wheel_1_LEFT_F" parent="body_left_F" xyz="0 0.0484063 -0.0583795" rpy="-6.12323e-17 -1.5708 0"/>
   <xacro:wheel name="wheel_2_LEFT_F" parent="body_left_F" xyz="0 1.07779e-16 -0.0583795" rpy="-6.12323e-17 -1.5708 0"/>
@@ -127,5 +153,5 @@
   <!-- RIGHT_F -->
   <xacro:body_right name="body_right_F" parent="RF_UPPER_LEG"
-                    xyz="0.19 -0.05 0" rpy="3.14159 0 1.5708"/>
+                    xyz="0.19 -0.05 0" rpy="3.14159 0 1.5708" ankle_center="${ankle_flat}"/>
   <xacro:wheel name="wheel_1_RIGHT_F" parent="body_right_F" xyz="2.08167e-17 0.0583795 0.0484062" rpy="-1.5708 0.992087 -1.5708"/>
   <xacro:wheel name="wheel_2_RIGHT_F" parent="body_right_F" xyz="0 0.0583795 1.10544e-16" rpy="-1.5708 0.967866 -1.5708"/>
@@ -134,5 +160,5 @@
   <!-- RIGHT_H -->
   <xacro:body_right name="body_right_H" parent="RH_UPPER_LEG"
-                    xyz="-0.19 -0.05 0" rpy="0 0 1.5708"/>
+                    xyz="-0.19 -0.05 0" rpy="0 0 1.5708" ankle_center="${-ankle_flat}"/>
   <xacro:wheel name="wheel_1_RIGHT_H" parent="body_right_H" xyz="2.08167e-17 0.0583795 0.0484062" rpy="-1.5708 0.992087 -1.5708"/>
   <xacro:wheel name="wheel_2_RIGHT_H" parent="body_right_H" xyz="0 0.0583795 1.10544e-16" rpy="-1.5708 0.967866 -1.5708"/>

File: src/mulinex_description/urdf/traquad.xacro (robot description, xacro)
@@ -119,25 +119,5 @@
         feet_type="$(arg feet_type)"
         />
-    <xacro:body_left  name="LH" parent="LH_UPPER_LEG" xyz="-0.19 0.05 0" rpy="1.5708 0 1.5708"/>
-    <xacro:body_left  name="LF" parent="LF_UPPER_LEG" xyz="0.19 0.05 0" rpy="-1.5708 0 1.5708"/>
-    <xacro:body_right name="RF" parent="RF_UPPER_LEG" xyz="0.19 -0.05 0" rpy="3.14159 0 1.5708"/>
-    <xacro:body_right name="RH" parent="RH_UPPER_LEG" xyz="-0.19 -0.05 0" rpy="0 0 1.5708"/>
-    <!-- Wheels for each body (4 per leg) -->
-    <xacro:wheel name="wheel_1_LH" parent="LH" xyz="0 0.0484 -0.0584" rpy="-6.12323e-17 -1.5708 0"/>
-    <xacro:wheel name="wheel_2_LH" parent="LH" xyz="0 1.07779e-16 -0.0584" rpy="-6.12323e-17 -1.5708 0"/>
-    <xacro:wheel name="wheel_3_LH" parent="LH" xyz="0 -0.05103 -0.0584" rpy="-6.12323e-17 -1.5708 0"/>
-    <xacro:wheel name="wheel_4_LH" parent="LH" xyz="0 -0.07668 -0.0417" rpy="-6.12323e-17 -1.5708 0"/>
-    <xacro:wheel name="wheel_1_LF" parent="LF" xyz="0 0.0484 -0.0584" rpy="-6.12323e-17 -1.5708 0"/>
-    <xacro:wheel name="wheel_2_LF" parent="LF" xyz="0 1.07779e-16 -0.0584" rpy="-6.12323e-17 -1.5708 0"/>
-    <xacro:wheel name="wheel_3_LF" parent="LF" xyz="0 -0.05103 -0.0584" rpy="-6.12323e-17 -1.5708 0"/>
-    <xacro:wheel name="wheel_4_LF" parent="LF" xyz="0 -0.07668 -0.0417" rpy="-6.12323e-17 -1.5708 0"/>
-    <xacro:wheel name="wheel_1_RF" parent="RF" xyz="2.08167e-17 0.05838 0.04841" rpy="-1.5708 0.992087 -1.5708"/>
-    <xacro:wheel name="wheel_2_RF" parent="RF" xyz="0 0.05838 1.10544e-16" rpy="-1.5708 0.967866 -1.5708"/>
-    <xacro:wheel name="wheel_3_RF" parent="RF" xyz="-2.08167e-17 0.05838 -0.05103" rpy="-1.5708 0.967866 -1.5708"/>
-    <xacro:wheel name="wheel_4_RF" parent="RF" xyz="-3.46945e-17 0.04174 -0.07668" rpy="-1.5708 0.992087 -1.5708"/>
-    <xacro:wheel name="wheel_1_RH" parent="RH" xyz="2.08167e-17 0.05838 0.04841" rpy="-1.5708 0.992087 -1.5708"/>
-    <xacro:wheel name="wheel_2_RH" parent="RH" xyz="0 0.05838 1.10544e-16" rpy="-1.5708 0.967866 -1.5708"/>
-    <xacro:wheel name="wheel_3_RH" parent="RH" xyz="-2.08167e-17 0.05838 -0.05103" rpy="-1.5708 0.967866 -1.5708"/>
-    <xacro:wheel name="wheel_4_RH" parent="RH" xyz="-3.46945e-17 0.04174 -0.07668" rpy="-1.5708 0.992087 -1.5708"/>
+    <!-- Track bodies and wheels are instantiated in track.xacro (included above) -->
     <xacro:imu_sensor namespace="$(arg mulinex_namespace)"/>
     <xacro:lidar_sensor tredi="$(arg lidar_3D)" namespace="$(arg mulinex_namespace)"/>

Commit message: Model track wheels with passive rollers
Replace the Gazebo-only anisotropic wheel friction with passive rollers,
so the lateral compliance of the tracks is a physical, URDF-standard
parameter that works the same in Gazebo and Isaac Sim.

- ground wheels (1-3 of each track): the driven hub carries 8 spherical
  rollers (r=8 mm, centres at 7 mm) on passive continuous joints whose
  axis is tangent to the rim; roller_damping tunes lateral resistance
- idler wheel (4): unchanged cylinder collision
- isotropic wheel friction mu=0.5 (Isaac Sim default)
- roller inertia raised to 1e-5 kg m^2: in DART the effective joint
  damping is capped at about inertia/timestep

Standard maneuver (w=0.5 rad/s in place, then v=0.2 m/s + w=0.5 rad/s):
roller_damping=1e-4 gives 92% / 85% of the commanded yaw rate with
0.018 m/s lateral drift; isotropic friction without rollers gives 0%.

File: src/mulinex_description/urdf/track.xacro (robot description, xacro)
@@ -7,8 +7,15 @@
   <xacro:property name="wheel_izz" default="1.15625e-05"/>
   <xacro:property name="wheel_mesh" default="file://$(find mulinex_description)/meshes//wheel.stl"/>
-  <!-- Gazebo-only wheel friction: reduced lateral friction lets the skid-steer tracks turn.
-       mu acts along fdir1 (= wheel axis, lateral), mu2 along the rolling direction. -->
-  <xacro:property name="wheel_mu_lat" value="0.1"/>
-  <xacro:property name="wheel_mu_long" value="1.0"/>
+  <!-- Wheel/roller contact. Isotropic friction (Isaac Sim default 0.5), lateral compliance
+       comes from passive rollers on the ground wheels: roller_damping tunes lateral resistance -->
+  <xacro:property name="wheel_mu" value="0.5"/>
+  <xacro:property name="roller_n" value="8"/>
+  <xacro:property name="roller_radius" value="0.008"/>
+  <xacro:property name="roller_ring_radius" value="0.007"/>
+  <xacro:property name="roller_mass" value="0.005"/>
+  <xacro:property name="roller_damping" value="1e-4"/>
+  <!-- roller rotational inertia (armature-like, larger than the physical 1.3e-7): in DART the
+       effective joint damping is capped at about inertia/timestep -->
+  <xacro:property name="roller_inertia" value="1e-5"/>
   <xacro:property name="body_mass" value="0.6"/>
   <!-- Passive ankle: range centred on the pose where the track lies flat
@@ -20,29 +27,86 @@
   <xacro:property name="body_right_mesh" default="file://$(find mulinex_description)/meshes//body_right.stl"/>
   <!-- ===================== MACRO ===================== -->
-  <!-- Macro RUOTA -->
-  <xacro:macro name="wheel" params="name parent xyz rpy">
-    <link name="${name}">
-      <inertial>
-        <origin xyz="0 0 -0.0225" rpy="0 0 0"/>
-        <mass value="${wheel_mass}"/>
-        <inertia ixx="${wheel_ixx}" ixy="0" ixz="0"
-                 iyy="${wheel_iyy}" iyz="0" izz="${wheel_izz}"/>
+  <xacro:macro name="contact_friction" params="link">
+    <gazebo reference="${link}">
+      <collision>
+        <surface>
+          <friction>
+            <ode>
+              <mu>${wheel_mu}</mu>
+              <mu2>${wheel_mu}</mu2>
+            </ode>
+          </friction>
+        </surface>
+      </collision>
+    </gazebo>
+  </xacro:macro>
+  <!-- Passive rollers on the wheel rim (wheel link frame, axis z, mid-plane z=-0.0225),
+       each roller axis tangent to the rim -->
+  <xacro:macro name="roller_ring" params="wheel k">
+    <xacro:property name="th" value="${2*pi*k/roller_n}"/>
+    <link name="${wheel}_roller_${k}">
+      <inertial>
+        <mass value="${roller_mass}"/>
+        <inertia ixx="${roller_inertia}" ixy="0" ixz="0" iyy="${roller_inertia}" iyz="0" izz="${roller_inertia}"/>
       </inertial>
       <visual>
-        <origin xyz="0 0 -0.045" rpy="-1.5708 -1.5708 0"/>
-        <geometry>
-          <mesh filename="${wheel_mesh}"/>
-        </geometry>
-        <material name="${name}_material">
-          <color rgba="0.615686 0.811765 0.929412 1"/>
+        <geometry>
+          <sphere radius="${roller_radius}"/>
+        </geometry>
+        <material name="roller_material">
+          <color rgba="0.3 0.3 0.3 1"/>
         </material>
       </visual>
       <collision>
-        <!-- primitive equivalent of wheel.stl (r=0.015, width=0.045), friction params are applied to it -->
+        <geometry>
+          <sphere radius="${roller_radius}"/>
+        </geometry>
+      </collision>
+    </link>
+    <joint name="${wheel}_roller_${k}_joint" type="continuous">
+      <origin xyz="${roller_ring_radius*cos(th)} ${roller_ring_radius*sin(th)} -0.0225" rpy="0 0 ${th + pi/2}"/>
+      <parent link="${wheel}"/>
+      <child link="${wheel}_roller_${k}"/>
+      <axis xyz="1 0 0"/>
+      <dynamics damping="${roller_damping}" friction="0.0"/>
+    </joint>
+    <xacro:contact_friction link="${wheel}_roller_${k}"/>
+    <xacro:if value="${k + 1 &lt; roller_n}">
+      <xacro:roller_ring wheel="${wheel}" k="${k + 1}"/>
+    </xacro:if>
+  </xacro:macro>
+  <!-- Macro RUOTA: rollers=true for ground wheels, false for the raised idler -->
+  <xacro:macro name="wheel" params="name parent xyz rpy rollers:=true">
+    <link name="${name}">
+      <xacro:if value="${rollers}">
+        <xacro:property name="hub_mass" value="${wheel_mass - roller_n*roller_mass}"/>
+      </xacro:if>
+      <xacro:unless value="${rollers}">
+        <xacro:property name="hub_mass" value="${wheel_mass}"/>
+      </xacro:unless>
+      <inertial>
         <origin xyz="0 0 -0.0225" rpy="0 0 0"/>
-        <geometry>
-          <cylinder radius="0.015" length="0.045"/>
-        </geometry>
-      </collision>
+        <mass value="${hub_mass}"/>
+        <inertia ixx="${wheel_ixx*hub_mass/wheel_mass}" ixy="0" ixz="0"
+                 iyy="${wheel_iyy*hub_mass/wheel_mass}" iyz="0" izz="${wheel_izz*hub_mass/wheel_mass}"/>
+      </inertial>
+      <xacro:unless value="${rollers}">
+        <visual>
+          <origin xyz="0 0 -0.045" rpy="-1.5708 -1.5708 0"/>
+          <geometry>
+            <mesh filename="${wheel_mesh}"/>
+          </geometry>
+          <material name="${name}_material">
+            <color rgba="0.615686 0.811765 0.929412 1"/>
+          </material>
+        </visual>
+        <collision>
+          <!-- primitive equivalent of wheel.stl (r=0.015, width=0.045) -->
+          <origin xyz="0 0 -0.0225" rpy="0 0 0"/>
+          <geometry>
+            <cylinder radius="0.015" length="0.045"/>
+          </geometry>
+        </collision>
+      </xacro:unless>
     </link>
     <joint name="joint_${name}" type="continuous">
@@ -53,18 +117,10 @@
       <limit effort="10" velocity="100000"/>
     </joint>
-    <gazebo reference="${name}">
-      <collision>
-        <surface>
-          <friction>
-            <ode>
-              <mu>${wheel_mu_lat}</mu>
-              <mu2>${wheel_mu_long}</mu2>
-              <!-- wheel axis (joint axis, link z) -->
-              <fdir1>0 0 1</fdir1>
-            </ode>
-          </friction>
-        </surface>
-      </collision>
-    </gazebo>
+    <xacro:if value="${rollers}">
+      <xacro:roller_ring wheel="${name}" k="0"/>
+    </xacro:if>
+    <xacro:unless value="${rollers}">
+      <xacro:contact_friction link="${name}"/>
+    </xacro:unless>
   </xacro:macro>
   <!-- Macro CORPO LEFT -->
@@ -143,5 +199,5 @@
   <xacro:wheel name="wheel_2_LEFT_H" parent="body_left_H" xyz="0 1.07779e-16 -0.0583795" rpy="-6.12323e-17 -1.5708 0"/>
   <xacro:wheel name="wheel_3_LEFT_H" parent="body_left_H" xyz="0 -0.0510313 -0.0583795" rpy="-6.12323e-17 -1.5708 0"/>
-  <xacro:wheel name="wheel_4_LEFT_H" parent="body_left_H" xyz="0 -0.0766777 -0.0417374" rpy="-6.12323e-17 -1.5708 0"/>
+  <xacro:wheel name="wheel_4_LEFT_H" parent="body_left_H" xyz="0 -0.0766777 -0.0417374" rpy="-6.12323e-17 -1.5708 0" rollers="false"/>
   <!-- LEFT_F -->
   <xacro:body_left name="body_left_F" parent="LF_UPPER_LEG"
@@ -150,5 +206,5 @@
   <xacro:wheel name="wheel_2_LEFT_F" parent="body_left_F" xyz="0 1.07779e-16 -0.0583795" rpy="-6.12323e-17 -1.5708 0"/>
   <xacro:wheel name="wheel_3_LEFT_F" parent="body_left_F" xyz="0 -0.0510313 -0.0583795" rpy="-6.12323e-17 -1.5708 0"/>
-  <xacro:wheel name="wheel_4_LEFT_F" parent="body_left_F" xyz="0 -0.0766777 -0.0417374" rpy="-6.12323e-17 -1.5708 0"/>
+  <xacro:wheel name="wheel_4_LEFT_F" parent="body_left_F" xyz="0 -0.0766777 -0.0417374" rpy="-6.12323e-17 -1.5708 0" rollers="false"/>
   <!-- RIGHT_F -->
   <xacro:body_right name="body_right_F" parent="RF_UPPER_LEG"
@@ -157,5 +213,5 @@
   <xacro:wheel name="wheel_2_RIGHT_F" parent="body_right_F" xyz="0 0.0583795 1.10544e-16" rpy="-1.5708 0.967866 -1.5708"/>
   <xacro:wheel name="wheel_3_RIGHT_F" parent="body_right_F" xyz="-2.08167e-17 0.0583795 -0.0510312" rpy="-1.5708 0.967866 -1.5708"/>
-  <xacro:wheel name="wheel_4_RIGHT_F" parent="body_right_F" xyz="-3.46945e-17 0.0417374 -0.0766777" rpy="-1.5708 0.992087 -1.5708"/>
+  <xacro:wheel name="wheel_4_RIGHT_F" parent="body_right_F" xyz="-3.46945e-17 0.0417374 -0.0766777" rpy="-1.5708 0.992087 -1.5708" rollers="false"/>
   <!-- RIGHT_H -->
   <xacro:body_right name="body_right_H" parent="RH_UPPER_LEG"
@@ -164,4 +220,4 @@
   <xacro:wheel name="wheel_2_RIGHT_H" parent="body_right_H" xyz="0 0.0583795 1.10544e-16" rpy="-1.5708 0.967866 -1.5708"/>
   <xacro:wheel name="wheel_3_RIGHT_H" parent="body_right_H" xyz="-2.08167e-17 0.0583795 -0.0510312" rpy="-1.5708 0.967866 -1.5708"/>
-  <xacro:wheel name="wheel_4_RIGHT_H" parent="body_right_H" xyz="-3.46945e-17 0.0417374 -0.0766777" rpy="-1.5708 0.992087 -1.5708"/>
+  <xacro:wheel name="wheel_4_RIGHT_H" parent="body_right_H" xyz="-3.46945e-17 0.0417374 -0.0766777" rpy="-1.5708 0.992087 -1.5708" rollers="false"/>
 </robot>

Commit message: Add visual track belt meshes
Add a visual-only rubber belt to each track, generated by
meshes/make_track_belt.py from the wheel positions and the ankle
structure mesh: the belt wraps the three roller wheels and the idler,
passes over the ankle structure and has rubber lugs on the outside.

The belt is attached as a second visual of body_left_* / body_right_*;
collisions and physics are unchanged (standard maneuver still gives
91% yaw rate in place and 86% while turning).

File: src/mulinex_description/urdf/track.xacro (robot description, xacro)
@@ -26,4 +26,7 @@
   <xacro:property name="body_left_mesh" default="file://$(find mulinex_description)/meshes//body_left.stl"/>
   <xacro:property name="body_right_mesh" default="file://$(find mulinex_description)/meshes//body_right.stl"/>
+  <!-- visual-only track belt wrapping the four wheels (generated by meshes/make_track_belt.py) -->
+  <xacro:property name="track_belt_left_mesh" value="file://$(find mulinex_description)/meshes//track_belt_left.stl"/>
+  <xacro:property name="track_belt_right_mesh" value="file://$(find mulinex_description)/meshes//track_belt_right.stl"/>
   <!-- ===================== MACRO ===================== -->
   <xacro:macro name="contact_friction" params="link">
@@ -150,4 +153,12 @@
         </material>
       </visual>
+      <visual>
+        <geometry>
+          <mesh filename="${track_belt_left_mesh}"/>
+        </geometry>
+        <material name="track_belt_material">
+          <color rgba="0.13 0.13 0.14 1"/>
+        </material>
+      </visual>
       <collision>
         <origin xyz="0 0 0" rpy="0 0 3.14159"/>
@@ -182,4 +193,12 @@
         <material name="${name}_material">
           <color rgba="0.647059 0.647059 0.647059 1"/>
+        </material>
+      </visual>
+      <visual>
+        <geometry>
+          <mesh filename="${track_belt_right_mesh}"/>
+        </geometry>
+        <material name="track_belt_material">
+          <color rgba="0.13 0.13 0.14 1"/>
         </material>
       </visual>
