Commit message: Set real robot masses and make traquad left/right symmetric
Masses (inertias scaled by the same factor):
- body 1.7 kg including IMU and lidar links (base_link 1.565 kg),
  each shoulder 0.6 kg, each upper leg 0.6 kg, each track 0.325 kg
  (track_mass_scale; body, wheels and rollers scaled proportionally);
  total 7.8 kg
- links.xacro: shoulder_mass_scale / upper_leg_mass_scale, default 1
  so the Mulinex models are unchanged

Left/right symmetry:
- base_link COM on y = 0, ixy = iyz = 0
- links.xacro: symmetric_left_right (default false, true in traquad):
  right shoulder/upper-leg inertials are the mirror of the left ones
  (COM z and ixz, iyz signs were wrong)
- right wheels mounted with the same phase as the left ones
  (rpy -1.5708 0 -1.5708 instead of 0.992/0.968 rad)

Effect in Isaac Sim: yaw rate in place is now the same in both
directions (rollers 98% / 98%), no spurious yaw when driving straight,
and the robot no longer spins when it lands in Gazebo.

File: src/mulinex_description/urdf/links.xacro (robot description, xacro)
@@ -18,4 +18,11 @@
     <xacro:property name="ANKLE_2_ROLL3_y" value="${58.0 * 0.001}" />
     <xacro:property name="PI" value="3.141592" />
+    <!-- mass scale factors of the shoulder (hip module) and upper-leg links: 1 for Mulinex,
+         set by robots that include this file before including it (e.g. traquad.xacro) -->
+    <xacro:property name="shoulder_mass_scale" default="1.0" />
+    <xacro:property name="upper_leg_mass_scale" default="1.0" />
+    <!-- true = right shoulder/upper-leg inertials are the exact mirror (y -> -y) of the left ones
+         (COM z and ixz, iyz signs); false keeps the original values (Mulinex) -->
+    <xacro:property name="symmetric_left_right" default="false" />
     <!-- MULINEX VISUALIZATION meshes -->
     <xacro:property name="mulinex_module_left_front"
@@ -204,12 +211,12 @@
             </collision>
             <inertial>
-                <mass value="0.47669673" />
+                <mass value="${0.47669673 * shoulder_mass_scale}" />
                 <xacro:if value="${prefix == 'LF'}">
                     <origin
                         xyz="7.2487360e-02 3.1582591e-02 -2.4812434e-03"
                         rpy="0 0 0" />
-                    <inertia ixx="2.1574269e-04" ixy="-3.3437484e-05"
-                        ixz="-2.4284668e-06" iyy="3.0607390e-03"
-                        iyz="-2.0388977e-06" izz="3.0504273e-03" />
+                    <inertia ixx="${2.1574269e-04 * shoulder_mass_scale}" ixy="${-3.3437484e-05 * shoulder_mass_scale}"
+                        ixz="${-2.4284668e-06 * shoulder_mass_scale}" iyy="${3.0607390e-03 * shoulder_mass_scale}"
+                        iyz="${-2.0388977e-06 * shoulder_mass_scale}" izz="${3.0504273e-03 * shoulder_mass_scale}" />
                 </xacro:if>
                 <xacro:if value="${prefix == 'LH'}">
@@ -217,23 +224,23 @@
                         xyz="-7.2487360e-02 3.1582591e-02 2.4812434e-03"
                         rpy="0 0 0" />
-                    <inertia ixx="2.1574269e-04" ixy="3.3437484e-05"
-                        ixz="-2.4284668e-06" iyy="3.0607390e-03"
-                        iyz="-2.0388977e-06" izz="3.0504273e-03" />
+                    <inertia ixx="${2.1574269e-04 * shoulder_mass_scale}" ixy="${3.3437484e-05 * shoulder_mass_scale}"
+                        ixz="${-2.4284668e-06 * shoulder_mass_scale}" iyy="${3.0607390e-03 * shoulder_mass_scale}"
+                        iyz="${-2.0388977e-06 * shoulder_mass_scale}" izz="${3.0504273e-03 * shoulder_mass_scale}" />
                 </xacro:if>
                 <xacro:if value="${prefix == 'RF'}">
                     <origin
-                        xyz="7.2487360e-02 -3.1582591e-02 2.4812434e-03"
+                        xyz="7.2487360e-02 -3.1582591e-02 ${-2.4812434e-03 if symmetric_left_right else 2.4812434e-03}"
                         rpy="0 0 0" />
-                    <inertia ixx="2.1574269e-04" ixy="3.3437484e-05"
-                        ixz="2.4284668e-06" iyy="3.0607390e-03"
-                        iyz="-2.0388977e-06" izz="3.0504273e-03" />
+                    <inertia ixx="${2.1574269e-04 * shoulder_mass_scale}" ixy="${3.3437484e-05 * shoulder_mass_scale}"
+                        ixz="${(-2.4284668e-06 if symmetric_left_right else 2.4284668e-06) * shoulder_mass_scale}" iyy="${3.0607390e-03 * shoulder_mass_scale}"
+                        iyz="${(2.0388977e-06 if symmetric_left_right else -2.0388977e-06) * shoulder_mass_scale}" izz="${3.0504273e-03 * shoulder_mass_scale}" />
                 </xacro:if>
                 <xacro:if value="${prefix == 'RH'}">
                     <origin
-                        xyz="-7.2487360e-02 -3.1582591e-02 -2.4812434e-03"
+                        xyz="-7.2487360e-02 -3.1582591e-02 ${2.4812434e-03 if symmetric_left_right else -2.4812434e-03}"
                         rpy="0 0 0" />
-                    <inertia ixx="2.1574269e-04" ixy="-3.3437484e-05"
-                        ixz="2.4284668e-06" iyy="3.0607390e-03"
-                        iyz="-2.0388977e-06" izz="3.0504273e-03" />
+                    <inertia ixx="${2.1574269e-04 * shoulder_mass_scale}" ixy="${-3.3437484e-05 * shoulder_mass_scale}"
+                        ixz="${(-2.4284668e-06 if symmetric_left_right else 2.4284668e-06) * shoulder_mass_scale}" iyy="${3.0607390e-03 * shoulder_mass_scale}"
+                        iyz="${(2.0388977e-06 if symmetric_left_right else -2.0388977e-06) * shoulder_mass_scale}" izz="${3.0504273e-03 * shoulder_mass_scale}" />
                 </xacro:if>
             </inertial>
@@ -380,12 +387,12 @@
             </collision>
             <inertial>
-                <mass value="0.47669673" />
+                <mass value="${0.47669673 * upper_leg_mass_scale}" />
                 <xacro:if value="${prefix == 'LF'}">
                     <origin
                         xyz="7.2487360e-02 3.1582591e-02 -2.4812434e-03"
                         rpy="0 0 0" />
-                    <inertia ixx="2.1574269e-04" ixy="-3.3437484e-05"
-                        ixz="-2.4284668e-06" iyy="3.0607390e-03"
-                        iyz="-2.0388977e-06" izz="3.0504273e-03" />
+                    <inertia ixx="${2.1574269e-04 * upper_leg_mass_scale}" ixy="${-3.3437484e-05 * upper_leg_mass_scale}"
+                        ixz="${-2.4284668e-06 * upper_leg_mass_scale}" iyy="${3.0607390e-03 * upper_leg_mass_scale}"
+                        iyz="${-2.0388977e-06 * upper_leg_mass_scale}" izz="${3.0504273e-03 * upper_leg_mass_scale}" />
                 </xacro:if>
                 <xacro:if value="${prefix == 'LH'}">
@@ -393,23 +400,23 @@
                         xyz="-7.2487360e-02 3.1582591e-02 2.4812434e-03"
                         rpy="0 0 0" />
-                    <inertia ixx="2.1574269e-04" ixy="3.3437484e-05"
-                        ixz="-2.4284668e-06" iyy="3.0607390e-03"
-                        iyz="-2.0388977e-06" izz="3.0504273e-03" />
+                    <inertia ixx="${2.1574269e-04 * upper_leg_mass_scale}" ixy="${3.3437484e-05 * upper_leg_mass_scale}"
+                        ixz="${-2.4284668e-06 * upper_leg_mass_scale}" iyy="${3.0607390e-03 * upper_leg_mass_scale}"
+                        iyz="${-2.0388977e-06 * upper_leg_mass_scale}" izz="${3.0504273e-03 * upper_leg_mass_scale}" />
                 </xacro:if>
                 <xacro:if value="${prefix == 'RF'}">
                     <origin
-                        xyz="7.2487360e-02 -3.1582591e-02 2.4812434e-03"
+                        xyz="7.2487360e-02 -3.1582591e-02 ${-2.4812434e-03 if symmetric_left_right else 2.4812434e-03}"
                         rpy="0 0 0" />
-                    <inertia ixx="2.1574269e-04" ixy="3.3437484e-05"
-                        ixz="2.4284668e-06" iyy="3.0607390e-03"
-                        iyz="-2.0388977e-06" izz="3.0504273e-03" />
+                    <inertia ixx="${2.1574269e-04 * upper_leg_mass_scale}" ixy="${3.3437484e-05 * upper_leg_mass_scale}"
+                        ixz="${(-2.4284668e-06 if symmetric_left_right else 2.4284668e-06) * upper_leg_mass_scale}" iyy="${3.0607390e-03 * upper_leg_mass_scale}"
+                        iyz="${(2.0388977e-06 if symmetric_left_right else -2.0388977e-06) * upper_leg_mass_scale}" izz="${3.0504273e-03 * upper_leg_mass_scale}" />
                 </xacro:if>
                 <xacro:if value="${prefix == 'RH'}">
                     <origin
-                        xyz="-7.2487360e-02 -3.1582591e-02 -2.4812434e-03"
+                        xyz="-7.2487360e-02 -3.1582591e-02 ${2.4812434e-03 if symmetric_left_right else -2.4812434e-03}"
                         rpy="0 0 0" />
-                    <inertia ixx="2.1574269e-04" ixy="-3.3437484e-05"
-                        ixz="2.4284668e-06" iyy="3.0607390e-03"
-                        iyz="-2.0388977e-06" izz="3.0504273e-03" />
+                    <inertia ixx="${2.1574269e-04 * upper_leg_mass_scale}" ixy="${-3.3437484e-05 * upper_leg_mass_scale}"
+                        ixz="${(-2.4284668e-06 if symmetric_left_right else 2.4284668e-06) * upper_leg_mass_scale}" iyy="${3.0607390e-03 * upper_leg_mass_scale}"
+                        iyz="${(2.0388977e-06 if symmetric_left_right else -2.0388977e-06) * upper_leg_mass_scale}" izz="${3.0504273e-03 * upper_leg_mass_scale}" />
                 </xacro:if>
             </inertial>

File: src/mulinex_description/urdf/track.xacro (robot description, xacro)
@@ -2,8 +2,11 @@
 <robot xmlns:xacro="http://ros.org/wiki/xacro" name="track">
   <!-- ===================== ARGOMENTI COMUNI ===================== -->
-  <xacro:property name="wheel_mass" default="0.1"/>
-  <xacro:property name="wheel_ixx" default="2.26562e-05"/>
-  <xacro:property name="wheel_iyy" default="2.26562e-05"/>
-  <xacro:property name="wheel_izz" default="1.15625e-05"/>
+  <!-- whole track (body + 4 wheels + rollers) = 1.0 kg x track_mass_scale = 0.325 kg (real robot);
+       masses and inertias of body, wheels and rollers are scaled by the same factor -->
+  <xacro:property name="track_mass_scale" default="0.325"/>
+  <xacro:property name="wheel_mass" default="${0.1 * track_mass_scale}"/>
+  <xacro:property name="wheel_ixx" default="${2.26562e-05 * track_mass_scale}"/>
+  <xacro:property name="wheel_iyy" default="${2.26562e-05 * track_mass_scale}"/>
+  <xacro:property name="wheel_izz" default="${1.15625e-05 * track_mass_scale}"/>
   <xacro:property name="wheel_mesh" default="file://$(find mulinex_description)/meshes//wheel.stl"/>
   <!-- Wheel/roller contact. Isotropic friction (Isaac Sim default 0.5), lateral compliance
@@ -13,10 +16,10 @@
   <xacro:property name="roller_radius" value="0.008"/>
   <xacro:property name="roller_ring_radius" value="0.007"/>
-  <xacro:property name="roller_mass" value="0.005"/>
+  <xacro:property name="roller_mass" value="${0.005 * track_mass_scale}"/>
   <xacro:property name="roller_damping" value="1e-4"/>
   <!-- roller rotational inertia (armature-like, larger than the physical 1.3e-7): in DART the
        effective joint damping is capped at about inertia/timestep -->
   <xacro:property name="roller_inertia" value="1e-5"/>
-  <xacro:property name="body_mass" value="0.6"/>
+  <xacro:property name="body_mass" value="${0.6 * track_mass_scale}"/>
   <!-- Passive ankle: range centred on the pose where the track lies flat
        (wheels 1-3 level) with HFE at init_pos (+-1.13 rad) -->
@@ -141,6 +144,6 @@
         <origin xyz="0.0238777 -0.00119624 -0.00412068" rpy="0 0 0"/>
         <mass value="${body_mass}"/>
-        <inertia ixx="0.000408384" ixy="6.93353e-06" ixz="3.09979e-05"
-                 iyy="0.000335218" iyz="-2.90084e-05" izz="0.000303698"/>
+        <inertia ixx="${0.000408384 * track_mass_scale}" ixy="${6.93353e-06 * track_mass_scale}" ixz="${3.09979e-05 * track_mass_scale}"
+                 iyy="${0.000335218 * track_mass_scale}" iyz="${-2.90084e-05 * track_mass_scale}" izz="${0.000303698 * track_mass_scale}"/>
       </inertial>
       <visual>
@@ -183,6 +186,6 @@
         <origin xyz="-0.0238777 0.00412068 -0.00119624" rpy="0 0 0"/>
         <mass value="${body_mass}"/>
-        <inertia ixx="0.000408384" ixy="3.09979e-05" ixz="-6.93353e-06"
-                 iyy="0.000303698" iyz="2.90084e-05" izz="0.000335218"/>
+        <inertia ixx="${0.000408384 * track_mass_scale}" ixy="${3.09979e-05 * track_mass_scale}" ixz="${-6.93353e-06 * track_mass_scale}"
+                 iyy="${0.000303698 * track_mass_scale}" iyz="${2.90084e-05 * track_mass_scale}" izz="${0.000335218 * track_mass_scale}"/>
       </inertial>
       <visual>
@@ -229,14 +232,14 @@
   <xacro:body_right name="body_right_F" parent="RF_UPPER_LEG"
                     xyz="0.19 -0.05 0" rpy="3.14159 0 1.5708" ankle_center="${ankle_flat}"/>
-  <xacro:wheel name="wheel_1_RIGHT_F" parent="body_right_F" xyz="2.08167e-17 0.0583795 0.0484062" rpy="-1.5708 0.992087 -1.5708"/>
-  <xacro:wheel name="wheel_2_RIGHT_F" parent="body_right_F" xyz="0 0.0583795 1.10544e-16" rpy="-1.5708 0.967866 -1.5708"/>
-  <xacro:wheel name="wheel_3_RIGHT_F" parent="body_right_F" xyz="-2.08167e-17 0.0583795 -0.0510312" rpy="-1.5708 0.967866 -1.5708"/>
-  <xacro:wheel name="wheel_4_RIGHT_F" parent="body_right_F" xyz="-3.46945e-17 0.0417374 -0.0766777" rpy="-1.5708 0.992087 -1.5708" rollers="false"/>
+  <xacro:wheel name="wheel_1_RIGHT_F" parent="body_right_F" xyz="2.08167e-17 0.0583795 0.0484062" rpy="-1.5708 0 -1.5708"/>
+  <xacro:wheel name="wheel_2_RIGHT_F" parent="body_right_F" xyz="0 0.0583795 1.10544e-16" rpy="-1.5708 0 -1.5708"/>
+  <xacro:wheel name="wheel_3_RIGHT_F" parent="body_right_F" xyz="-2.08167e-17 0.0583795 -0.0510312" rpy="-1.5708 0 -1.5708"/>
+  <xacro:wheel name="wheel_4_RIGHT_F" parent="body_right_F" xyz="-3.46945e-17 0.0417374 -0.0766777" rpy="-1.5708 0 -1.5708" rollers="false"/>
   <!-- RIGHT_H -->
   <xacro:body_right name="body_right_H" parent="RH_UPPER_LEG"
                     xyz="-0.19 -0.05 0" rpy="0 0 1.5708" ankle_center="${-ankle_flat}"/>
-  <xacro:wheel name="wheel_1_RIGHT_H" parent="body_right_H" xyz="2.08167e-17 0.0583795 0.0484062" rpy="-1.5708 0.992087 -1.5708"/>
-  <xacro:wheel name="wheel_2_RIGHT_H" parent="body_right_H" xyz="0 0.0583795 1.10544e-16" rpy="-1.5708 0.967866 -1.5708"/>
-  <xacro:wheel name="wheel_3_RIGHT_H" parent="body_right_H" xyz="-2.08167e-17 0.0583795 -0.0510312" rpy="-1.5708 0.967866 -1.5708"/>
-  <xacro:wheel name="wheel_4_RIGHT_H" parent="body_right_H" xyz="-3.46945e-17 0.0417374 -0.0766777" rpy="-1.5708 0.992087 -1.5708" rollers="false"/>
+  <xacro:wheel name="wheel_1_RIGHT_H" parent="body_right_H" xyz="2.08167e-17 0.0583795 0.0484062" rpy="-1.5708 0 -1.5708"/>
+  <xacro:wheel name="wheel_2_RIGHT_H" parent="body_right_H" xyz="0 0.0583795 1.10544e-16" rpy="-1.5708 0 -1.5708"/>
+  <xacro:wheel name="wheel_3_RIGHT_H" parent="body_right_H" xyz="-2.08167e-17 0.0583795 -0.0510312" rpy="-1.5708 0 -1.5708"/>
+  <xacro:wheel name="wheel_4_RIGHT_H" parent="body_right_H" xyz="-3.46945e-17 0.0417374 -0.0766777" rpy="-1.5708 0 -1.5708" rollers="false"/>
 </robot>

File: src/mulinex_description/urdf/traquad.xacro (robot description, xacro)
@@ -15,4 +15,14 @@
             simplify_meshes="${simplify_meshes}"/>
     </xacro:macro>
+    <!-- ===================== MASSES (real robot) =====================
+         body 1.7 kg including IMU (0.010 kg) and lidar (0.125 kg) links, so base_link = 1.565 kg;
+         each shoulder 0.6 kg (body + 4 shoulders = 4.1 kg), each upper leg 0.6 kg,
+         each track 0.325 kg (track_mass_scale in track.xacro); total 7.8 kg. Inertias scale with the mass. -->
+    <xacro:property name="base_mass" value="${1.7 - 0.010 - 0.125}" />
+    <xacro:property name="base_mass_scale" value="${base_mass / 1.3008737}" />
+    <xacro:property name="shoulder_mass_scale" value="${0.6 / 0.47669673}" />
+    <xacro:property name="upper_leg_mass_scale" value="${0.6 / 0.47669673}" />
+    <!-- the robot is symmetric left/right, right legs mirror the left ones, base COM on y = 0 -->
+    <xacro:property name="symmetric_left_right" value="true" />
     <!-- Vi consiglio di creare xacro con i track e lo includete qui -->
     <xacro:include filename="$(find mulinex_description)/urdf/links.xacro" />
@@ -60,9 +70,11 @@
         </collision>
         <inertial>
-            <mass value="1.3008737" />
-            <origin xyz="-1.4565496e-03 -2.5110071e-03 -4.2484136e-03" rpy="0 0 0" />
-            <inertia ixx="4.0762590e-03" ixy="-2.5234809e-05" ixz="-3.2587794e-06"
-                iyy="9.2413606e-03" iyz="-8.0660183e-06"
-                izz="1.2268730e-02" />
+            <mass value="${base_mass}" />
+            <!-- left/right symmetric, COM on y = 0 and ixy = iyz = 0 -->
+            <origin xyz="-1.4565496e-03 0.0 -4.2484136e-03" rpy="0 0 0" />
+            <inertia ixx="${4.0762590e-03 * base_mass_scale}" ixy="0.0"
+                ixz="${-3.2587794e-06 * base_mass_scale}"
+                iyy="${9.2413606e-03 * base_mass_scale}" iyz="0.0"
+                izz="${1.2268730e-02 * base_mass_scale}" />
         </inertial>
     </link>
